Commit message: Imported upstream version '5.1.3' of 'upstream'

File: tiago_description/urdf/arm/arm.urdf.xacro (robot description, xacro)
@@ -49,5 +49,6 @@
         <origin xyz="0 0 0" rpy="0 0 0" />
         <geometry>
-          <mesh filename="package://tiago_description/meshes/arm/arm_1.stl" scale="1 ${-1 * tiago_dual} ${reflect}"/>
+          <!-- TODO Remove reflected meshes https://github.com/gazebosim/ros_gz/issues/587 -->
+          <mesh filename="package://tiago_description/meshes/arm/arm_1${'_dual' if tiago_dual == 1 else ''}${'_reflected' if reflect == -1 else ''}.stl" scale="1 1 1"/>
         </geometry>
         <material name="White"/>
@@ -56,5 +57,5 @@
         <origin xyz="0 0 0" rpy="0 0 0" />
         <geometry>
-          <mesh filename="package://tiago_description/meshes/arm/arm_1_collision.dae" scale="1 ${-1 * tiago_dual} ${reflect}"/>
+          <mesh filename="package://tiago_description/meshes/arm/arm_1_collision${'_dual' if tiago_dual == 1 else ''}${'_reflected' if reflect == -1 else ''}.stl" scale="1 1 1"/>
         </geometry>
       </collision>
@@ -81,5 +82,5 @@
         <origin xyz="0 0 0" rpy="${0 * deg_to_rad} ${0 * deg_to_rad} ${0 * deg_to_rad}" />
         <geometry>
-          <mesh filename="package://tiago_description/meshes/arm/arm_2.stl" scale="1 1 ${reflect}"/>
+          <mesh filename="package://tiago_description/meshes/arm/arm_2${'_reflected' if reflect == -1 else ''}.stl" scale="1 1 1"/>
         </geometry>
         <material name="DarkGrey" />
@@ -89,5 +90,5 @@
         <origin xyz="0 0 0" rpy="${0 * deg_to_rad} ${0 * deg_to_rad} ${0 * deg_to_rad}" />
         <geometry>
-          <mesh filename="package://tiago_description/meshes/arm/arm_2_collision.dae" scale="1 1 ${reflect}"/>
+          <mesh filename="package://tiago_description/meshes/arm/arm_2_collision${'_reflected' if reflect == -1 else ''}.stl" scale="1 1 1"/>
         </geometry>
       </collision>
@@ -113,5 +114,5 @@
         <origin xyz="0 0 0" rpy="0 0 0" />
         <geometry>
-          <mesh filename="package://tiago_description/meshes/arm/arm_3.stl" scale="1 1 ${reflect}"/>
+          <mesh filename="package://tiago_description/meshes/arm/arm_3${'_reflected' if reflect == -1 else ''}.stl" scale="1 1 1"/>
         </geometry>
         <material name="DarkGrey" />
@@ -120,5 +121,5 @@
         <origin xyz="0 0 0" rpy="0 0 0" />
         <geometry>
-          <mesh filename="package://tiago_description/meshes/arm/arm_3_collision.dae" scale="1 1 ${reflect}"/>
+          <mesh filename="package://tiago_description/meshes/arm/arm_3_collision${'_reflected' if reflect == -1 else ''}.stl" scale="1 1 1"/>
         </geometry>
       </collision>
@@ -127,5 +128,5 @@
       <parent link="${name}_2_link" />
       <child link="${name}_3_link" />
-      <origin xyz="0.0895 0.0 -0.0015" rpy="${-90.0 * deg_to_rad} ${(90.0 - reflect * 90.0) * deg_to_rad} ${reflect * 90.0 * deg_to_rad}"/>
+      <origin xyz="0.0895 0.0 ${reflect * 0.0015}" rpy="${-90.0 * deg_to_rad} ${(90.0 - reflect * 90.0) * deg_to_rad} ${reflect * 90.0 * deg_to_rad}"/>
       <axis xyz="0 0 1" />
       <xacro:property name="arm_3_lower_limit" value="${-45. if tiago_dual == 1 else -202.5}"/>
@@ -145,5 +146,5 @@
         <origin xyz="0 0 0" rpy="0 0 0" />
         <geometry>
-          <mesh filename="package://tiago_description/meshes/arm/arm_4.stl" scale="${reflect} ${reflect} ${reflect}"/>
+          <mesh filename="package://tiago_description/meshes/arm/arm_4${'_reflected' if reflect == -1 else ''}.stl" scale="1 1 1"/>
         </geometry>
         <material name="DarkGrey" />
@@ -152,5 +153,5 @@
         <origin xyz="0 0 0" rpy="0 0 0" />
         <geometry>
-          <mesh filename="package://tiago_description/meshes/arm/arm_4_collision.dae" scale="${reflect} ${reflect} ${reflect}"/>
+          <mesh filename="package://tiago_description/meshes/arm/arm_4_collision${'_reflected' if reflect == -1 else ''}.stl" scale="1 1 1"/>
         </geometry>
       </collision>
